Commit message: s

File: urdf/ackermann_bot.xacro (robot description, xacro)
@@ -10,5 +10,4 @@
   <xacro:property name="chassis_height" value="0.2"/>
   <!-- Plugins -->
-  <xacro:include filename="$(find xacro)/gazebo/gazebo.xacro"/>
   <!-- Base Link -->
   <link name="base_link">

File: urdf/my_bot_core.xacro (robot description, xacro)
@@ -1,175 +1,205 @@
-<?xml version="1.0" ?>
+<?xml version="1.0"?>
 <robot xmlns:xacro="http://www.ros.org/wiki/xacro">
-  <link name="base_link"/>
-  <material name="Gray"><color rgba="0.5 0.5 0.5 1.0"/></material>
-  <material name="Black"><color rgba="0.0 0.0 0.0 1.0"/></material>
-  <material name="Red"><color rgba="1.0 0.0 0.0 1.0"/></material>
-  <material name="Blue"><color rgba="0.0 0.0 1.0 1.0"/></material>
-  <material name="Green"><color rgba="0.0 1.0 0.0 1.0"/></material>
-  <material name="White"><color rgba="1.0 1.0 1.0 1.0"/></material>
+  <material name="Gray">
+    <color rgba="0.5 0.5 0.5 1.0" />
+  </material>
+  <material name="Black">
+    <color rgba="0.0 0.0 0.0 1.0" />
+  </material>
+  <link name="base_link">
+  </link>
+  <joint name="base_footprint_joint" type="fixed">
+    <parent link="base_link" />
+    <child link="base_footprint" />
+    <origin xyz="0 0 0" rpy="0 0 0" />
+  </joint>
+  <link name="base_footprint">
+  </link>
   <!-- Chassis -->
   <link name="chassis">
     <inertial>
-      <mass value="1.0"/>
-      <origin rpy="0 0 0" xyz="0 0 0"/>
-      <inertia ixx="0.060833" ixy="0" ixz="0" iyy="0.1275" iyz="0" izz="0.173333"/>
-    </inertial>
-    <visual>
-      <origin rpy="0 0 0" xyz="0 0 0"/>
-      <geometry><box size="1.2 0.8 0.3"/></geometry>
-      <material name="Gray"/>
-    </visual>
-    <collision>
-      <origin rpy="0 0 0" xyz="0 0 0"/>
-      <geometry><box size="1.2 0.8 0.3"/></geometry>
-    </collision>
-  </link>
-  <joint name="base_to_chassis" type="fixed">
-    <parent link="base_link"/>
-    <child link="chassis"/>
-    <origin rpy="0 0 0" xyz="0 0 0.15"/>
-  </joint>
-  <!-- DRIVETRAIN -->
-  <!-- Steering Wheel -->
+      <mass value="1.0" />
+      <origin rpy="0 0 0" xyz="0 0 0" />
+      <inertia ixx="0.060833" ixy="0" ixz="0" iyy="0.1275" iyz="0" izz="0.173333" />
+    </inertial>
+    <visual>
+      <origin rpy="0 0 0" xyz="0 0 0" />
+      <geometry>
+        <box size="1.2 0.8 0.3" />
+      </geometry>
+      <material name="Gray" />
+    </visual>
+    <collision>
+      <origin rpy="0 0 0" xyz="0 0 0" />
+      <geometry>
+        <box size="1.2 0.8 0.3" />
+      </geometry>
+    </collision>
+  </link>
+  <joint name="chassis_joint" type="fixed">
+    <parent link="base_link" />
+    <child link="chassis" />
+    <origin rpy="0 0 0" xyz="0 0 0.15" />
+  </joint>
+  <gazebo reference="chassis">
+    <material>Gazebo/White</material>
+  </gazebo>
+<!-- Steering Wheel -->
   <link name="steering_wheel_link">
     <inertial>
-      <mass value="0.5"/>
-      <origin rpy="0 0 0" xyz="0 0 0"/>
-      <inertia ixx="0.001" ixy="0" ixz="0" iyy="0.001" iyz="0" izz="0.001"/>
-    </inertial>
-    <visual>
-      <origin rpy="0 0 0" xyz="0 0 0"/>
-      <geometry><cylinder radius="0.1" length="0.02"/></geometry>
-      <material name="Black"/>
+      <mass value="0.5" />
+      <origin rpy="0 0 0" xyz="0 0 0" />
+      <inertia ixx="0.001" ixy="0" ixz="0" iyy="0.001" iyz="0" izz="0.001" />
+    </inertial>
+    <visual>
+      <origin rpy="0 0 0" xyz="0 0 0" />
+      <geometry>
+        <cylinder radius="0.1" length="0.02" />
+      </geometry>
+      <material name="Black" />
     </visual>
   </link>
   <joint name="steering_wheel_joint" type="revolute">
-    <parent link="chassis"/>
-    <child link="steering_wheel_link"/>
-    <origin rpy="0 0 0" xyz="0.3 0 0.2"/>
-    <axis xyz="0 0 1"/>
-    <limit effort="100" velocity="10" lower="-7.85" upper="7.85"/>
-  </joint>
-  <!-- Front Left Steering -->
+    <parent link="chassis" />
+    <child link="steering_wheel_link" />
+    <origin rpy="0 0 0" xyz="0.3 0 0.2" />
+    <axis xyz="0 0 1" />
+    <limit effort="100" velocity="10" lower="-7.85" upper="7.85" />
+  </joint>
+  <!-- Steering Mechanism -->
   <link name="front_left_steering">
     <inertial>
-      <mass value="0.1"/>
-      <origin rpy="0 0 0" xyz="0 0 0"/>
-      <inertia ixx="0.001" ixy="0" ixz="0" iyy="0.001" iyz="0" izz="0.001"/>
+      <mass value="0.1" />
+      <origin rpy="0 0 0" xyz="0 0 0" />
+      <inertia ixx="0.001" ixy="0" ixz="0" iyy="0.001" iyz="0" izz="0.001" />
+    </inertial>
+  </link>
+  <link name="front_right_steering">
+    <inertial>
+      <mass value="0.1" />
+      <origin rpy="0 0 0" xyz="0 0 0" />
+      <inertia ixx="0.001" ixy="0" ixz="0" iyy="0.001" iyz="0" izz="0.001" />
     </inertial>
   </link>
   <joint name="front_left_steering_joint" type="revolute">
-    <parent link="chassis"/>
-    <child link="front_left_steering"/>
-    <origin rpy="0 0 0" xyz="0.4533 0.46 -0.15"/>
-    <axis xyz="0 0 1"/>
-    <limit effort="100" velocity="10" lower="-0.5" upper="0.5"/>
+    <parent link="chassis" />
+    <child link="front_left_steering" />
+    <origin rpy="0 0 0" xyz="0.4533 0.46 -0.15" />
+    <axis xyz="0 0 1" />
+    <limit effort="100" velocity="10" lower="-0.5" upper="0.5" />
+  </joint>
+  <joint name="front_right_steering_joint" type="revolute">
+    <parent link="chassis" />
+    <child link="front_right_steering" />
+    <origin rpy="0 0 0" xyz="0.4533 -0.46 -0.15" />
+    <axis xyz="0 0 1" />
+    <limit effort="100" velocity="10" lower="-0.5" upper="0.5" />
+    <mimic joint="front_left_steering_joint" multiplier="-1" offset="0" />
   </joint>
   <!-- Front Left Wheel -->
   <link name="front_left_wheel">
     <inertial>
-      <mass value="0.5"/>
-      <origin rpy="1.5708 0 0" xyz="0 0 0"/>
-      <inertia ixx="0.00665" ixy="0" ixz="0" iyy="0.00665" iyz="0" izz="0.0121"/>
-    </inertial>
-    <visual>
-      <origin rpy="1.5708 0 0" xyz="0 0 0"/>
-      <geometry><cylinder length="0.12" radius="0.22"/></geometry>
-      <material name="Black"/>
-    </visual>
-    <collision>
-      <origin rpy="1.5708 0 0" xyz="0 0 0"/>
-      <geometry><cylinder length="0.12" radius="0.22"/></geometry>
+      <mass value="0.5" />
+      <origin rpy="1.5708 0 0" xyz="0 0 0" />
+      <inertia ixx="0.00665" ixy="0" ixz="0" iyy="0.00665" iyz="0" izz="0.0121" />
+    </inertial>
+    <visual>
+      <origin rpy="1.5708 0 0" xyz="0 0 0" />
+      <geometry>
+        <cylinder length="0.12" radius="0.22" />
+      </geometry>
+      <material name="Black" />
+    </visual>
+    <collision>
+      <origin rpy="1.5708 0 0" xyz="0 0 0" />
+      <geometry>
+        <cylinder length="0.12" radius="0.22" />
+      </geometry>
     </collision>
   </link>
   <joint name="front_left_wheel_joint" type="continuous">
-    <parent link="front_left_steering"/>
-    <child link="front_left_wheel"/>
-    <origin rpy="0 0 0" xyz="0 0 0"/>
-    <axis xyz="0 1 0"/>
-  </joint>
-  <!-- Front Right Steering -->
-  <link name="front_right_steering">
-    <inertial>
-      <mass value="0.1"/>
-      <origin rpy="0 0 0" xyz="0 0 0"/>
-      <inertia ixx="0.001" ixy="0" ixz="0" iyy="0.001" iyz="0" izz="0.001"/>
-    </inertial>
-  </link>
-  <joint name="front_right_steering_joint" type="revolute">
-    <parent link="chassis"/>
-    <child link="front_right_steering"/>
-    <origin rpy="0 0 0" xyz="0.4533 -0.46 -0.15"/>
-    <axis xyz="0 0 1"/>
-    <limit effort="100" velocity="10" lower="-0.5" upper="0.5"/>
-    <mimic joint="front_left_steering_joint" multiplier="-1" offset="0"/>
+    <parent link="front_left_steering" />
+    <child link="front_left_wheel" />
+    <origin rpy="0 0 0" xyz="0 0 0" />
+    <axis xyz="0 1 0" />
   </joint>
   <!-- Front Right Wheel -->
   <link name="front_right_wheel">
     <inertial>
-      <mass value="0.5"/>
-      <origin rpy="1.5708 0 0" xyz="0 0 0"/>
-      <inertia ixx="0.00665" ixy="0" ixz="0" iyy="0.00665" iyz="0" izz="0.0121"/>
-    </inertial>
-    <visual>
-      <origin rpy="1.5708 0 0" xyz="0 0 0"/>
-      <geometry><cylinder length="0.12" radius="0.22"/></geometry>
-      <material name="Black"/>
-    </visual>
-    <collision>
-      <origin rpy="1.5708 0 0" xyz="0 0 0"/>
-      <geometry><cylinder length="0.12" radius="0.22"/></geometry>
+      <mass value="0.5" />
+      <origin rpy="1.5708 0 0" xyz="0 0 0" />
+      <inertia ixx="0.00665" ixy="0" ixz="0" iyy="0.00665" iyz="0" izz="0.0121" />
+    </inertial>
+    <visual>
+      <origin rpy="1.5708 0 0" xyz="0 0 0" />
+      <geometry>
+        <cylinder length="0.12" radius="0.22" />
+      </geometry>
+      <material name="Black" />
+    </visual>
+    <collision>
+      <origin rpy="1.5708 0 0" xyz="0 0 0" />
+      <geometry>
+        <cylinder length="0.12" radius="0.22" />
+      </geometry>
     </collision>
   </link>
   <joint name="front_right_wheel_joint" type="continuous">
-    <parent link="front_right_steering"/>
-    <child link="front_right_wheel"/>
-    <origin rpy="0 0 0" xyz="0 0 0"/>
-    <axis xyz="0 1 0"/>
+    <parent link="front_right_steering" />
+    <child link="front_right_wheel" />
+    <origin rpy="0 0 0" xyz="0 0 0" />
+    <axis xyz="0 1 0" />
   </joint>
   <!-- Rear Wheels -->
   <link name="rear_left_wheel">
     <inertial>
-      <mass value="0.5"/>
-      <origin rpy="1.5708 0 0" xyz="0 0 0"/>
-      <inertia ixx="0.00665" ixy="0" ixz="0" iyy="0.00665" iyz="0" izz="0.0121"/>
-    </inertial>
-    <visual>
-      <origin rpy="1.5708 0 0" xyz="0 0 0"/>
-      <geometry><cylinder length="0.12" radius="0.22"/></geometry>
-      <material name="Black"/>
-    </visual>
-    <collision>
-      <origin rpy="1.5708 0 0" xyz="0 0 0"/>
-      <geometry><cylinder length="0.12" radius="0.22"/></geometry>
+      <mass value="0.5" />
+      <origin rpy="1.5708 0 0" xyz="0 0 0" />
+      <inertia ixx="0.00665" ixy="0" ixz="0" iyy="0.00665" iyz="0" izz="0.0121" />
+    </inertial>
+    <visual>
+      <origin rpy="1.5708 0 0" xyz="0 0 0" />
+      <geometry>
+        <cylinder length="0.12" radius="0.22" />
+      </geometry>
+      <material name="Black" />
+    </visual>
+    <collision>
+      <origin rpy="1.5708 0 0" xyz="0 0 0" />
+      <geometry>
+        <cylinder length="0.12" radius="0.22" />
+      </geometry>
     </collision>
   </link>
   <joint name="rear_left_wheel_joint" type="continuous">
-    <parent link="chassis"/>
-    <child link="rear_left_wheel"/>
-    <origin rpy="0 0 0" xyz="-0.4533  0.46 -0.15"/>
-    <axis xyz="0 1 0"/>
+    <parent link="chassis" />
+    <child link="rear_left_wheel" />
+    <origin rpy="0 0 0" xyz="-0.4533  0.46 -0.15" />
+    <axis xyz="0 1 0" />
   </joint>
   <link name="rear_right_wheel">
     <inertial>
-      <mass value="0.5"/>
-      <origin rpy="1.5708 0 0" xyz="0 0 0"/>
-      <inertia ixx="0.00665" ixy="0" ixz="0" iyy="0.00665" iyz="0" izz="0.0121"/>
-    </inertial>
-    <visual>
-      <origin rpy="1.5708 0 0" xyz="0 0 0"/>
-      <geometry><cylinder length="0.12" radius="0.22"/></geometry>
-      <material name="Black"/>
-    </visual>
-    <collision>
-      <origin rpy="1.5708 0 0" xyz="0 0 0"/>
-      <geometry><cylinder length="0.12" radius="0.22"/></geometry>
+      <mass value="0.5" />
+      <origin rpy="1.5708 0 0" xyz="0 0 0" />
+      <inertia ixx="0.00665" ixy="0" ixz="0" iyy="0.00665" iyz="0" izz="0.0121" />
+    </inertial>
+    <visual>
+      <origin rpy="1.5708 0 0" xyz="0 0 0" />
+      <geometry>
+        <cylinder length="0.12" radius="0.22" />
+      </geometry> <material name="Black" />
+    </visual>
+    <collision>
+      <origin rpy="1.5708 0 0" xyz="0 0 0" />
+      <geometry>
+        <cylinder length="0.12" radius="0.22" />
+      </geometry>
     </collision>
   </link>
   <joint name="rear_right_wheel_joint" type="continuous">
-    <parent link="chassis"/>
-    <child link="rear_right_wheel"/>
-    <origin rpy="0 0 0" xyz="-0.4533 -0.46 -0.15"/>
-    <axis xyz="0 1 0"/>
+    <parent link="chassis" />
+    <child link="rear_right_wheel" />
+    <origin rpy="0 0 0" xyz="-0.4533 -0.46 -0.15" />
+    <axis xyz="0 1 0" />
   </joint>
 </robot>

File: urdf/my_bot_gazebo_control.xacro (robot description, xacro)
@@ -3,11 +3,4 @@
   <gazebo>
     <plugin name='ackermann_drive_controller' filename='libgazebo_ros_ackermann_drive.so'>
-      <ros>
-        <namespace>demo</namespace>
-        <remapping>cmd_vel:=cmd_demo</remapping>
-        <remapping>odom:=odom_demo</remapping>
-        <remapping>distance:=distance_demo</remapping>
-        <remapping>steerangle:=steerangle_demo</remapping>
-      </ros>
       <update_rate>100.0</update_rate>
       <!-- wheels -->
@@ -25,12 +18,5 @@
       <max_steering_angle>7.85</max_steering_angle>
       <!-- Max absolute linear speed in m/s -->
-      <max_speed>20</max_speed>
-      <!-- PID tuning -->
-      <left_steering_pid_gain>1500 0 1</left_steering_pid_gain>
-      <left_steering_i_range>0 0</left_steering_i_range>
-      <right_steering_pid_gain>1500 0 1</right_steering_pid_gain>
-      <right_steering_i_range>0 0</right_steering_i_range>
-      <linear_velocity_pid_gain>1000 0 1</linear_velocity_pid_gain>
-      <linear_velocity_i_range>0 0</linear_velocity_i_range>
+      <max_speed>200</max_speed>
       <!-- output -->
       <publish_odom>true</publish_odom>
@@ -39,6 +25,6 @@
       <publish_distance>true</publish_distance>
       <publish_steerangle>true</publish_steerangle>
-      <odometry_frame>odom_demo</odometry_frame>
-      <robot_base_frame>chassis</robot_base_frame>
+      <odometry_frame>odom</odometry_frame>
+      <robot_base_frame>base_link</robot_base_frame>
     </plugin>
   </gazebo>
