Commit message: s

File: urdf/my_bot_core.xacro (robot description, xacro)
@@ -45,5 +45,5 @@
     <material>Gazebo/White</material>
   </gazebo>
-<!-- Steering Wheel -->
+  <!-- Steering Wheel -->
   <link name="steering_wheel_link">
     <inertial>
@@ -74,4 +74,11 @@
       <inertia ixx="0.001" ixy="0" ixz="0" iyy="0.001" iyz="0" izz="0.001" />
     </inertial>
+    <visual>
+      <origin rpy="0 0 0" xyz="0 0 0" />
+      <geometry>
+        <cylinder radius="0.1" length="0.02" />
+      </geometry>
+      <material name="Black" />
+    </visual>
   </link>
   <link name="front_right_steering">
@@ -81,4 +88,11 @@
       <inertia ixx="0.001" ixy="0" ixz="0" iyy="0.001" iyz="0" izz="0.001" />
     </inertial>
+    <visual>
+      <origin rpy="0 0 0" xyz="0 0 0" />
+      <geometry>
+        <cylinder radius="0.1" length="0.02" />
+      </geometry>
+      <material name="Black" />
+    </visual>
   </link>
   <joint name="front_left_steering_joint" type="revolute">
@@ -93,5 +107,5 @@
     <child link="front_right_steering" />
     <origin rpy="0 0 0" xyz="0.4533 -0.46 -0.15" />
-    <axis xyz="0 0 1" />
+    <axis xyz="0 0 -1" />
     <limit effort="100" velocity="10" lower="-0.5" upper="0.5" />
     <mimic joint="front_left_steering_joint" multiplier="-1" offset="0" />
@@ -188,5 +202,6 @@
       <geometry>
         <cylinder length="0.12" radius="0.22" />
-      </geometry> <material name="Black" />
+      </geometry>
+      <material name="Black" />
     </visual>
     <collision>
