Commit message: s

File: urdf/lidar.xacro (robot description, xacro)
@@ -22,7 +22,7 @@
   </link>
   <joint name="lidar_joint" type="fixed">
-    <parent link="chassis_link" />
+    <parent link="base_link" />
     <child link="lidar" />
-    <origin rpy="0 0 0" xyz="0 0 0.19" />
+    <origin rpy="0 0 0" xyz="0 0 0.3455" />
   </joint>
   <gazebo reference="lidar">
