Commit message: s

File: urdf/my_bot_gazebo_control.xacro (robot description, xacro)
@@ -1,31 +1,134 @@
 <?xml version="1.0"?>
 <robot xmlns:xacro="http://www.ros.org/wiki/xacro">
-  <gazebo>
-    <plugin name='ackermann_drive_controller' filename='libgazebo_ros_ackermann_drive.so'>
-      <update_rate>100.0</update_rate>
-      <!-- wheels -->
-      <front_left_joint>front_left_wheel_joint</front_left_joint>
-      <front_right_joint>front_right_wheel_joint</front_right_joint>
-      <rear_left_joint>rear_left_wheel_joint</rear_left_joint>
-      <rear_right_joint>rear_right_wheel_joint</rear_right_joint>
-      <left_steering_joint>front_left_steering_joint</left_steering_joint>
-      <right_steering_joint>front_right_steering_joint</right_steering_joint>
-      <steering_wheel_joint>steering_wheel_joint</steering_wheel_joint>
-      <!-- Max absolute steer angle for tyre in radians-->
-      <!-- Any cmd_vel angular z greater than this would be capped -->
-      <max_steer>0.6458</max_steer>
-      <!-- Max absolute steering angle of steering wheel -->
-      <max_steering_angle>7.85</max_steering_angle>
-      <!-- Max absolute linear speed in m/s -->
-      <max_speed>200</max_speed>
-      <!-- output -->
-      <publish_odom>true</publish_odom>
-      <publish_odom_tf>true</publish_odom_tf>
-      <publish_wheel_tf>true</publish_wheel_tf>
-      <publish_distance>true</publish_distance>
-      <publish_steerangle>true</publish_steerangle>
-      <odometry_frame>odom</odometry_frame>
-      <robot_base_frame>base_link</robot_base_frame>
-    </plugin>
-  </gazebo>
+    <!-- GAZEBO COLOUR -->
+    <!-- Gazebo is unable to use the same <material> tags that are already in the URDF (that RViz
+    uses). -->
+    <!-- Instead, we need to add gazebo tags for our links that refer to Gazebo materials -->
+    <gazebo reference="chassis_link">
+        <material>Gazebo/White</material>
+        <mu1>0.5</mu1>
+        <mu2>0.5</mu2>
+    </gazebo>
+    <gazebo reference="fr_left_wheel_link">
+        <material>Gazebo/Grey</material>
+        <mu1>1.0</mu1>
+        <mu2>1.0</mu2>
+    </gazebo>
+    <gazebo reference="fr_right_wheel_link">
+        <material>Gazebo/Grey</material>
+        <mu1>1.0</mu1>
+        <mu2>1.0</mu2>
+    </gazebo>
+    <gazebo reference="re_left_wheel_link">
+        <material>Gazebo/Grey</material>
+        <mu1>1.0</mu1>
+        <mu2>1.0</mu2>
+    </gazebo>
+    <gazebo reference="re_right_wheel_link">
+        <material>Gazebo/Grey</material>
+        <mu1>1.0</mu1>
+        <mu2>1.0</mu2>
+    </gazebo>
+    <gazebo reference="virtual_steer_link">
+        <material>Gazebo/Yellow</material>
+    </gazebo>
+    <!-- JOINT STATE PUBLISHER -->
+    <!-- Gazebo requires the use of plugins to interact with other systems such as ROS. -->
+    <!-- This plugin will publish the joint_states for the selected joints
+            (which robot_state_publisher can then use to broadcast the approprate tf).
+         Using Gazebo ROS2 control plugin (ros2_control) (part of ROS2 control system) publishing and
+    control of joint.-->
+    <gazebo>
+        <plugin name="gazebo_ros_joint_state_publisher"
+            filename="libgazebo_ros_joint_state_publisher.so">
+            <update_rate>100</update_rate>
+            <joint_name>fr_right_steer_joint</joint_name>
+            <joint_name>fr_right_wheel_joint</joint_name>
+            <joint_name>fr_left_steer_joint</joint_name>
+            <joint_name>fr_left_wheel_joint</joint_name>
+            <joint_name>re_right_wheel_joint</joint_name>
+            <joint_name>re_left_wheel_joint</joint_name>
+            <joint_name>virtual_steering_wheel_joint</joint_name>
+        </plugin>
+    </gazebo>
+    <!-- This plugin will read a JointTrajectory message from the /set_joint_trajectory topic
+            and move the machine accordingly. It's a bit clunky but it works. -->
+    <!-- You'll probably want to add damping to the joints to stop them it flopping around.
+            e.g. <dynamics damping="10.0" friction="10.0"/> -->
+    <!-- Here's an example message to publish to test it:
+            ros2 topic pub -1 /set_joint_trajectory trajectory_msgs/msg/JointTrajectory  '{header: {frame_id:
+    world}, joint_names: [slider_joint, arm_joint], points: [  {positions: {0.8,0.6}} ]}' -->
+    <gazebo>
+        <plugin name="gazebo_ros_joint_pose_trajectory"
+            filename="libgazebo_ros_joint_pose_trajectory.so">
+            <update_rate>2</update_rate>
+        </plugin>
+    </gazebo>
+    <!-- ACKERMANN DRIVE PLUGIN -->
+    <gazebo>
+        <plugin name='gazebo_ackermann_drive' filename='libgazebo_ros_ackermann_drive.so'>
+            <ros>
+                <!-- <namespace>ugv_gazebo_ackermann</namespace> -->
+                <remapping>cmd_vel:=cmd_vel</remapping>
+                <remapping>odom:=odom/bot</remapping>
+                <remapping>distance:=distance/bot</remapping>
+            </ros>
+            <update_rate>100.0</update_rate>
+            <!-- wheels -->
+            <front_left_joint>fr_left_wheel_joint</front_left_joint>
+            <front_right_joint>fr_right_wheel_joint</front_right_joint>
+            <rear_left_joint>re_left_wheel_joint</rear_left_joint>
+            <rear_right_joint>re_right_wheel_joint</rear_right_joint>
+            <left_steering_joint>fr_left_steer_joint</left_steering_joint>
+            <right_steering_joint>fr_right_steer_joint</right_steering_joint>
+            <steering_wheel_joint>virtual_steering_wheel_joint</steering_wheel_joint>
+            <!-- Max absolute steer angle for tyre in radians-->
+            <!-- Any cmd_vel angular z greater than this would be capped -->
+            <max_steer>0.383972</max_steer>
+            <!-- Max absolute steering angle of steering wheel -->
+            <max_steering_angle>1.570796</max_steering_angle>
+            <!-- Max absolute linear speed in m/s -->
+            <max_speed>5</max_speed>
+            <!-- PID tuning -->
+            <left_steering_pid_gain>1500 0 1</left_steering_pid_gain>
+            <left_steering_i_range>0 0</left_steering_i_range>
+            <right_steering_pid_gain>1500 0 1</right_steering_pid_gain>
+            <right_steering_i_range>0 0</right_steering_i_range>
+            <linear_velocity_pid_gain>1500 0 1</linear_velocity_pid_gain>
+            <linear_velocity_i_range>0 0</linear_velocity_i_range>
+            <!-- output -->
+            <publish_odom>true</publish_odom>
+            <publish_odom_tf>true</publish_odom_tf>     <!-- Don't pubslish this when using robot
+            localization -->
+            <publish_wheel_tf>false</publish_wheel_tf>  <!-- Don't publish this. It will override all
+            wheel frames to robot_base_frame parameter below.-->
+            <publish_distance>true</publish_distance>
+            <odometry_frame>odom</odometry_frame>
+            <robot_base_frame>base_footprint</robot_base_frame>
+        </plugin>
+    </gazebo>
+    <!-- Virtual Steering wheel -->
+    <link name="virtual_steer_link">
+        <visual>
+            <origin xyz="0.0 0.0 0.0" rpy="0.0 0.0 0.0" />
+            <geometry>
+                <box size="0.01 0.15 0.075" />
+            </geometry>
+            <material name="">
+                <color rgba="1.0 1.0 0.0 1" />
+            </material>
+        </visual>
+        <inertial>  <!-- Gazebo won't show this link without this inertial mass -->
+            <origin xyz="0.0 0.0 0.0" rpy="0.0 0.0 0.0" />
+            <mass value="0.001" />
+            <inertia ixx="0.0" ixy="0.0" ixz="0.0" iyy="0.0" iyz="0.0" izz="0.0" />
+        </inertial>
+    </link>
+    <joint name="virtual_steering_wheel_joint" type="revolute">
+        <origin xyz="-0.32 0.0 0.0" rpy="0.0 0.0 0.0" />
+        <parent link="chassis_link" />
+        <child link="virtual_steer_link" />
+        <axis xyz="-1 0 0" />
+        <limit lower="-3" upper="3" effort="200" velocity="20" />
+    </joint>
 </robot>

Commit message: s

File: urdf/camera1.xacro (robot description, xacro)
@@ -30,7 +30,7 @@
     <parent link="camera" />
     <child link="camera_optical" />
-    <origin rpy="-1.5708 0 -1.5708" xyz="0 0 0" />
+    <origin rpy="0 0 0" xyz="0 0 0" />
   </joint>
-  <gazebo reference="camera_link">
+  <gazebo reference="camera_optical">
     <material>Gazebo/Red</material>
     <sensor name="camera" type="camera">
@@ -51,5 +51,5 @@
       </camera>
       <plugin name="camera_controller" filename="libgazebo_ros_camera.so">
-        <frame_name>camera_link_optical</frame_name>
+        <frame_name>camera_optical</frame_name>
       </plugin>
     </sensor>

File: urdf/lidar.xacro (robot description, xacro)
@@ -26,5 +26,5 @@
     <origin rpy="0 0 0" xyz="0 0 0.19" />
   </joint>
-  <gazebo reference="laser_frame">
+  <gazebo reference="lidar">
     <material>Gazebo/Red</material>
     <sensor name="laser" type="ray">
@@ -50,5 +50,5 @@
         </ros>
         <output_type>sensor_msgs/LaserScan</output_type>
-        <frame_name>laser_frame</frame_name>
+        <frame_name>lidar</frame_name>
       </plugin>
     </sensor>

File: urdf/my_bot_core.xacro (robot description, xacro)
@@ -9,15 +9,26 @@
     <xacro:property name="wheel_mass" value="3.0" />
     <xacro:property name="steering_mass" value="0.01" />
+    <material name="white">
+        <color rgba="1 1 1 1" />
+    </material>
+    <material name="orange">
+        <color rgba="1 0.3 0.1 1"/>
+    </material>
+    <material name="blue">
+        <color rgba="0.2 0.2 1 1"/>
+    </material>
+    <material name="black">
+        <color rgba="0 0 0 1"/>
+    </material>
     <!-- BASE -->
+    <link name="base_link">
+    </link>
+    <joint name="base_joint" type="fixed">
+        <parent link="base_link" />
+        <child link="base_footprint" />
+        <origin xyz="0 0 0" rpy="0 0 0" />
+    </joint>
     <link name="base_footprint">
-            <origin xyz="0 0 0" rpy="0 0 0" />
-    </link>
-    <link name="base_link">
-    </link>
-    <joint name="base_joint" type="fixed">
-        <parent link="base_footprint" />
-        <child link="base_link" />
-        <origin xyz="0.0 0.0 0.0" rpy="0 0 0" />
-    </joint>
+    </link>
     <link name="chassis_link">
         <inertial>
@@ -34,4 +45,5 @@
                 <box size="1.2 0.8 0.3" />
             </geometry>
+            <material name="white"/>
         </visual>
         <collision>

File: urdf/my_bot_gazebo_control.xacro (robot description, xacro)
@@ -71,6 +71,6 @@
                 <!-- <namespace>ugv_gazebo_ackermann</namespace> -->
                 <remapping>cmd_vel:=cmd_vel</remapping>
-                <remapping>odom:=odom/bot</remapping>
-                <remapping>distance:=distance/bot</remapping>
+                <remapping>odom:=odom</remapping>
+                <remapping>distance:=distance</remapping>
             </ros>
             <update_rate>100.0</update_rate>
@@ -105,5 +105,5 @@
             <publish_distance>true</publish_distance>
             <odometry_frame>odom</odometry_frame>
-            <robot_base_frame>base_footprint</robot_base_frame>
+            <robot_base_frame>base_link</robot_base_frame>
         </plugin>
     </gazebo>

Commit message: Added experiment modes and evaluation setup

File: urdf/camera1.xacro (robot description, xacro)
@@ -12,5 +12,7 @@
         <box size="0.08 0.2 0.08" />
       </geometry>
-      <material name="Blue" />
+      <material name="Blue">
+        <color rgba="0.0 0.0 1.0 1.0" />
+      </material>
     </visual>
     <collision>

File: urdf/lidar.xacro (robot description, xacro)
@@ -12,5 +12,7 @@
         <cylinder length="0.08" radius="0.1" />
       </geometry>
-      <material name="Red" />
+      <material name="Red">
+        <color rgba="1.0 0.0 0.0 1.0" />
+      </material>
     </visual>
     <collision>
